Commit message: Control de manipulador movil

File: integracion_kuka_omni/robots/mpo_500/mpo_500.urdf.xacro (robot description, xacro)
@@ -2,12 +2,12 @@
 <robot name="mpo_500" xmlns:xacro="http://www.ros.org/wiki/xacro">
   <!--GAZEBO REFERENCES -->
-  <xacro:include filename="$(find neo_description)/robots/mpo_500/xacros/mpo_500_gazebo.xacro" />
+  <xacro:include filename="$(find integracion_kuka_omni)/robots/mpo_500/xacros/mpo_500_gazebo.xacro" />
   <!-- BODY -->
-  <xacro:include filename="$(find neo_description)/robots/mpo_500/xacros/mpo_500_body.xacro" />
-  <xacro:include filename="$(find kuka_kr4_description)/urdf/kuka_kr4.xacro" />
+  <xacro:include filename="$(find integracion_kuka_omni)/robots/mpo_500/xacros/mpo_500_body.xacro" />
+  <xacro:include filename="$(find kuka_kr4_description)/urdf/kuka_kr4_macro.xacro" />
   <!-- WHEELS -->
-  <xacro:include filename="$(find neo_description)/robots/mpo_500/xacros/omni_wheel.xacro" />
+  <xacro:include filename="$(find integracion_kuka_omni)/robots/mpo_500/xacros/omni_wheel.xacro" />
   <!-- SENSORS -->
-  <xacro:include filename="$(find neo_description)/robots/mpo_500/xacros/sick_laser.xacro" />
+  <xacro:include filename="$(find integracion_kuka_omni)/robots/mpo_500/xacros/sick_laser.xacro" />
   <link name="dummy">
    </link>

File: integracion_kuka_omni/robots/mpo_500/xacros/omni_wheel.xacro (robot description, xacro)
@@ -2,5 +2,5 @@
 <robot xmlns:xacro="http://www.ros.org/wiki/xacro" name="mpo_500">
   <xacro:macro name="omni_wheel_250" params="name parent *origin">
-   <joint name="${name}_joint" type="fixed">
+   <joint name="${name}_joint" type="continuous">
     <insert_block name="origin" />
     <axis xyz="0 1 0" />
